Commit message: Add the fixed model for the 3f gripper; this won't allow any feedback in rviz, but it will satisfy MoveIt's requirements to have a completely-defined robot state.

File: robotiq_3f_gripper_visualization/urdf/robotiq_3f.urdf.xacro (robot description, xacro)
@@ -1,9 +1,15 @@
 <?xml version="1.0"?>
 <robot xmlns:xacro="http://www.ros.org/wiki/xacro" name="s_model_open">
-    <xacro:macro name="robotiq_3f" params="parent prefix ">
+    <xacro:macro name="robotiq_3f" params="parent prefix *origin">
         <!-- mount the Gripper to the robot -->
-        <joint name="${prefix}_s_model_adapter" type="fixed" >
+        <link name="${prefix}s_model_base_link" />
+        <joint name="${prefix}s_model_base_joint" type="fixed">
+            <parent link="${parent}" />
+            <child link="${prefix}s_model_base_link" />
+            <xacro:insert_block name="origin" />
+        </joint>
+        <joint name="${prefix}s_model_adapter" type="fixed" >
             <origin xyz="0.0 0.0 0.015" rpy="0.0 0.0 0.0"/>
-	    <parent link="${parent}" />
+	          <parent link="${prefix}s_model_base_link" />
             <child link="${prefix}s_model_adapter_link" />
         </joint>

File: robotiq_3f_gripper_visualization/urdf/robotiq_3f_model.urdf.xacro (robot description, xacro)
@@ -2,5 +2,7 @@
 <robot xmlns:xacro="http://www.ros.org/wiki/xacro" name="s_model_open">
   <xacro:include filename="$(find robotiq_3f_gripper_visualization)/urdf/robotiq_3f.urdf.xacro" />
-  <xacro:robotiq_3f prefix="" parent="base_link"/>
+  <xacro:robotiq_3f prefix="" parent="base_link">
+    <origin xyz="0 0 0" rpy="0 0 0" />
+  </xacro:robotiq_3f>
   <link name="base_link" />
 </robot>
