Commit message: Use convex hull for collision

File: robotiq_hande_gripper_visualization/urdf/robotiq_hande.urdf.xacro (robot description, xacro)
@@ -44,7 +44,7 @@
       </visual>
       <collision>
-        <origin rpy="0 0 0" xyz="-0.0285 0 0.023"/>
+        <origin rpy="0 0 0" xyz="0 0 0"/>
         <geometry>
-          <box size="0.007 0.02 0.046"/>
+          <mesh filename="package://robotiq_hande_gripper_visualization/meshes/finger_1_collision.dae" scale="0.001 0.001 0.001"/>
         </geometry>
       </collision>
@@ -70,7 +70,7 @@
       </visual>
       <collision>
-        <origin rpy="0 0 0" xyz="0.0285 0 0.023"/>
+        <origin rpy="0 0 0" xyz="0 0 0"/>
         <geometry>
-          <box size="0.007 0.02 0.046"/>
+          <mesh filename="package://robotiq_hande_gripper_visualization/meshes/finger_2_collision.dae" scale="0.001 0.001 0.001"/>
         </geometry>
       </collision>
